Commit message: update smg_minitip

File: smg_gym/assets/robot_assets/smg_minitip/smg_tactip.urdf (robot description, URDF)
Before this commit: robot smart_grasping_sandbox, 27 links, 26 joints
Links:
- added link pivot_point_link, mass 0.0; visual sphere radius=0.005
- link F1_tcp_link: geometry visual sphere radius=0.001
- link F2_tcp_link: geometry visual sphere radius=0.001
- link F3_tcp_link: geometry visual sphere radius=0.001
Joints:
- added joint pivot_point_joint: type fixed, parent SMG_base_link, child pivot_point_link, origin xyz=0.0 0.0 0.25 rpy=0 0 0
- joint F1_tcp_joint: origin xyz=0.0 -0.02 0.052 rpy=0 0 0 -> xyz=0.0 -0.02 0.0535 rpy=0 0 0
- joint F2_tcp_joint: origin xyz=0.0 -0.02 0.052 rpy=0 0 0 -> xyz=0.0 -0.02 0.0535 rpy=0 0 0
- joint F3_tcp_joint: origin xyz=0.0 -0.02 0.052 rpy=0 0 0 -> xyz=0.0 -0.02 0.0535 rpy=0 0 0

Commit message: working pivot example but bug on reset

File: smg_gym/assets/robot_assets/smg_minitip/smg_tactip.urdf (robot description, URDF)
Before this commit: robot smart_grasping_sandbox, 28 links, 27 joints
Joints:
- joint pivot_point_joint: origin xyz=0.0 0.0 0.25 rpy=0 0 0 -> xyz=0.0 0.0 0.25 rpy=0.0 0.0 0.0

Commit message: PD control almost working in both. Working on rich contacts

File: smg_gym/assets/robot_assets/smg_minitip/smg_tactip.urdf (robot description, URDF)
Before this commit: robot smart_grasping_sandbox, 28 links, 27 joints
Joints:
- joint SMG_F1J1: limit lower=-0.785398163397 upper=0.785398163397 effort=50 velocity=1.0 -> lower=-0.785398163397 upper=0.785398163397 effort=1000 velocity=1000
- joint SMG_F1J2: limit lower=-1.3962634016 upper=1.0471975512 effort=50 velocity=1.0 -> lower=-1.3962634016 upper=1.0471975512 effort=1000 velocity=1000
- joint SMG_F1J3: limit lower=-1.0471975512 upper=1.57079632679 effort=50 velocity=1.0 -> lower=-1.0471975512 upper=1.3962634016 effort=1000 velocity=1000
- joint SMG_F2J1: limit lower=-0.785398163397 upper=0.785398163397 effort=30 velocity=1.0 -> lower=-0.785398163397 upper=0.785398163397 effort=1000 velocity=1000
- joint SMG_F2J2: limit lower=-1.3962634016 upper=1.0471975512 effort=30 velocity=1.0 -> lower=-1.3962634016 upper=1.0471975512 effort=1000 velocity=1000
- joint SMG_F2J3: limit lower=-1.0471975512 upper=1.57079632679 effort=30 velocity=1.0 -> lower=-1.0471975512 upper=1.3962634016 effort=1000 velocity=1000
- joint SMG_F3J1: limit lower=-0.785398163397 upper=0.785398163397 effort=30 velocity=1.0 -> lower=-0.785398163397 upper=0.785398163397 effort=1000 velocity=1000
- joint SMG_F3J2: limit lower=-1.3962634016 upper=1.0471975512 effort=30 velocity=1.0 -> lower=-1.3962634016 upper=1.0471975512 effort=1000 velocity=1000
- joint SMG_F3J3: limit lower=-1.0471975512 upper=1.57079632679 effort=30 velocity=1.0 -> lower=-1.0471975512 upper=1.3962634016 effort=1000 velocity=1000

Commit message: add n_stack and for observations and run a few experiments

File: smg_gym/assets/robot_assets/smg_minitip/smg_tactip.urdf (robot description, URDF)
Before this commit: robot smart_grasping_sandbox, 28 links, 27 joints
Joints:
- joint SMG_F1_tactip_tip_joint: origin (none) -> xyz=0.0 0.0 0.0535 rpy=1.57 0 0
- joint SMG_F2_tactip_tip_joint: origin (none) -> xyz=0.0 0.0 0.0535 rpy=1.57 0 0
- joint SMG_F3_tactip_tip_joint: origin (none) -> xyz=0.0 0.0 0.0535 rpy=1.57 0 0
