Commit message: adjust friction and other properties to more closely align with real

File: smg_gym/assets/object_assets/box.urdf (robot description, URDF)
Before this commit: robot cube, 1 links, 0 joints
Links:
- removed link cube
- added link box, mass 0.087; collision box size=.075 .075 .075; visual box size=.075 .075 .075
