Commit message: fix active_quat bug, struggling with true asym learning now

File: smg_gym/assets/robot_assets/smg_minitip_v2/smg_tactip_with_tip_targets.urdf (robot description, URDF)
Before this commit: robot smart_grasping_sandbox, 28 links, 27 joints
Links:
- added link F1_target_link, mass 0.0; collision mesh filename=tip/smg_tactip_target.stl; visual mesh filename=tip/smg_tactip_target.stl
- added link F2_target_link, mass 0.0; collision mesh filename=tip/smg_tactip_target.stl; visual mesh filename=tip/smg_tactip_target.stl
Joints:
- added joint F1_target_joint: type fixed, parent SMG_F1_tactip_body, child F1_target_link, origin xyz=0.0 -0.013 0.0575 rpy=0 0 0
- added joint F2_target_joint: type fixed, parent SMG_F2_tactip_body, child F2_target_link, origin xyz=0.0 -0.013 0.0575 rpy=0 0 0
- joint F3_target_joint: origin xyz=0.0 -0.0125 0.0575 rpy=0 0 0 -> xyz=0.0 -0.013 0.0575 rpy=0 0 0
