Commit message: update urdfs

File: smg_gym/assets/robot_assets/smg_minitip_v2/smg_tactip.urdf (robot description, URDF)
Before this commit: robot smart_grasping_sandbox, 27 links, 26 joints
Links:
- link SMG_F1_tactip_body: mass 0.01 -> 0.05
- link SMG_F2_tactip_body: mass 0.01 -> 0.05
- link SMG_F3_tactip_body: mass 0.01 -> 0.05
Joints:
- joint F1_tcp_joint: origin xyz=0.0 -0.0325 0.0575 rpy=0 0 0 -> xyz=0.0 -0.0325 0.0575 rpy=1.57 0 0
- joint F2_tcp_joint: origin xyz=0.0 -0.0325 0.0575 rpy=0 0 0 -> xyz=0.0 -0.0325 0.0575 rpy=1.57 0 0
- joint F3_tcp_joint: origin xyz=0.0 -0.0325 0.0575 rpy=0 0 0 -> xyz=0.0 -0.0325 0.0575 rpy=1.57 0 0

Commit message: switch to primitive object

File: smg_gym/assets/robot_assets/smg_minitip_v2/smg_tactip.urdf (robot description, URDF)
Before this commit: robot smart_grasping_sandbox, 27 links, 26 joints
Links:
- link SMG_F1_tactip_tip: geometry collision sphere radius=0.02; visual mesh filename=tip/smg_tactip_skin.obj
- link SMG_F2_tactip_tip: geometry collision sphere radius=0.02; visual mesh filename=tip/smg_tactip_skin.obj
- link SMG_F3_tactip_tip: geometry collision sphere radius=0.02; visual mesh filename=tip/smg_tactip_skin.obj

Commit message: update control to better match real proprio

File: smg_gym/assets/robot_assets/smg_minitip_v2/smg_tactip.urdf (robot description, URDF)
Before this commit: robot smart_grasping_sandbox, 27 links, 26 joints
Links:
- link SMG_F1_link_2: mass 0.0468986964963515 -> 0.071
- link SMG_F2_link_2: mass 0.0468986964963515 -> 0.071
- link SMG_F3_link_2: mass 0.0468986964963515 -> 0.071

Commit message: add onnx export of weights (not working yet)

File: smg_gym/assets/robot_assets/smg_minitip_v2/smg_tactip.urdf (robot description, URDF)
Before this commit: robot smart_grasping_sandbox, 27 links, 26 joints
Joints:
- joint pivot_point_joint: origin xyz=0.0 0.0 0.25 rpy=0.0 0.0 0.0 -> xyz=0.0 -0.016 0.25 rpy=0.0 0.0 0.0
