Commit message: modified generating grasp code to make grasp generation successful with allegro hand. Fixed bug regarding digitac collision and random ranges.

File: smg_gym/assets/robot_assets/allegro_hora/allegro_digitac.urdf (robot description, URDF)
Before this commit: robot allegro_hand_right, 33 links, 32 joints
Links:
- added link pivot_point_link, mass 0.0; visual sphere radius=0.005
- link digitac_body_link_11: geometry collision mesh filename=digitac/standard_digitac/digitac_asmb/meshes/digitac_body.o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; visual mesh filename=digitac/standard_digitac/digitac_asmb/meshes/digitac_body.o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
- link digitac_body_link_15: geometry collision mesh filename=digitac/standard_digitac/digitac_asmb/meshes/digitac_body.o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; visual mesh filename=digitac/standard_digitac/digitac_asmb/meshes/digitac_body.o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
- link digitac_body_link_3: geometry collision mesh filename=digitac/standard_digitac/digitac_asmb/meshes/digitac_body.o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; visual mesh filename=digitac/standard_digitac/digitac_asmb/meshes/digitac_body.o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
- link digitac_body_link_7: geometry collision mesh filename=digitac/standard_digitac/digitac_asmb/meshes/digitac_body.o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; visual mesh filename=digitac/standard_digitac/digitac_asmb/meshes/digitac_body.o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
- link digitac_tip_link_11: geometry collision mesh filename=digitac/standard_digitac/digitac_asmb_hollow/meshes/digitac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; visual mesh filename=digitac/standard_digitac/digitac_asmb_hollow/meshes/digitac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
- link digitac_tip_link_15: geometry collision mesh filename=digitac/standard_digitac/digitac_asmb_hollow/meshes/digitac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; visual mesh filename=digitac/standard_digitac/digitac_asmb_hollow/meshes/digitac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
- link digitac_tip_link_3: geometry collision mesh filename=digitac/standard_digitac/digitac_asmb_hollow/meshes/digitac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; visual mesh filename=digitac/standard_digitac/digitac_asmb_hollow/meshes/digitac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
- link digitac_tip_link_7: geometry collision mesh filename=digitac/standard_digitac/digitac_asmb_hollow/meshes/digitac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; visual mesh filename=digitac/standard_digitac/digitac_asmb_hollow/meshes/digitac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
Joints:
- added joint pivot_point_joint: type fixed, parent base_link, child pivot_point_link, origin xyz=0.25 0.0 0.0 rpy=-1.57 0.0 -1.57
- joint joint_0.0: limit lower=-0.47 upper=0.47 effort=0.35 velocity=6.283 -> lower=-0.47 upper=0.47 effort=10 velocity=6.283
- joint joint_1.0: limit lower=-0.196 upper=1.61 effort=0.35 velocity=6.283 -> lower=-0.196 upper=1.61 effort=10 velocity=6.283
- joint joint_10.0: limit lower=-0.174 upper=1.709 effort=0.35 velocity=6.283 -> lower=-0.174 upper=1.709 effort=10 velocity=6.283
- joint joint_11.0: limit lower=-0.227 upper=1.618 effort=0.35 velocity=6.283 -> lower=-0.227 upper=1.618 effort=10 velocity=6.283
- joint joint_12.0: limit lower=0.263 upper=1.396 effort=0.35 velocity=6.283 -> lower=0.263 upper=1.396 effort=10 velocity=6.283
- joint joint_13.0: limit lower=-0.105 upper=1.163 effort=0.35 velocity=6.283 -> lower=-0.105 upper=1.163 effort=10 velocity=6.283
- joint joint_14.0: limit lower=-0.189 upper=1.644 effort=0.35 velocity=6.283 -> lower=-0.189 upper=1.644 effort=10 velocity=6.283
- joint joint_15.0: limit lower=-0.162 upper=1.719 effort=0.35 velocity=6.283 -> lower=-0.162 upper=1.719 effort=10 velocity=6.283
- joint joint_2.0: limit lower=-0.174 upper=1.709 effort=0.35 velocity=6.283 -> lower=-0.174 upper=1.709 effort=10 velocity=6.283
- joint joint_3.0: limit lower=-0.227 upper=1.618 effort=0.35 velocity=6.283 -> lower=-0.227 upper=1.618 effort=10 velocity=6.283
- joint joint_4.0: limit lower=-0.47 upper=0.47 effort=0.35 velocity=6.283 -> lower=-0.47 upper=0.47 effort=10 velocity=6.283
- joint joint_5.0: limit lower=-0.196 upper=1.61 effort=0.35 velocity=6.283 -> lower=-0.196 upper=1.61 effort=10 velocity=6.283
- joint joint_6.0: limit lower=-0.174 upper=1.709 effort=0.35 velocity=6.283 -> lower=-0.174 upper=1.709 effort=10 velocity=6.283
- joint joint_7.0: limit lower=-0.227 upper=1.618 effort=0.35 velocity=6.283 -> lower=-0.227 upper=1.618 effort=10 velocity=6.283
- joint joint_8.0: limit lower=-0.47 upper=0.47 effort=0.35 velocity=6.283 -> lower=-0.47 upper=0.47 effort=10 velocity=6.283
- joint joint_9.0: limit lower=-0.196 upper=1.61 effort=0.35 velocity=6.283 -> lower=-0.196 upper=1.61 effort=10 velocity=6.283
